File: PCB/BottomPCB/BottomPCB.kicad_pcb (KiCad board)
At the start: 2 copper layers, 91.4 x 72.4 mm, 14 parts

Commit message: Updated PCB, 3d Models, and some Code to fix mistakes.
Parts:
- moved REF** 38.8 mm to (83.3, 52.1)
- moved REF** 38.8 mm to (144.2, 52.1)
- moved REF** 38.8 mm to (155.7, 100.3)
- moved REF** 38.8 mm to (108.7, 76.2)
- moved REF** 38.8 mm to (74.4, 100.3)
- moved REF** 38.8 mm to (74.4, 45.7)
- moved REF** 38.8 mm to (108.7, 106.7)
- moved REF** 38.8 mm to (93.5, 109.2)
- moved REF** 38.8 mm to (116.3, 45.7)
- moved REF** 38.8 mm to (136.6, 106.7)
- moved REF** 38.8 mm to (155.7, 45.7)
- moved REF** 38.8 mm to (121.4, 76.2)
- moved REF** 38.8 mm to (121.4, 106.7)
- moved REF** 38.8 mm to (115.0, 106.7)
Routing:
- net (no net): track 903.1 -> 900.6 mm
