File: PCB/TopPCB/TopPCB.kicad_pcb (KiCad board)
At the start: 2 copper layers, 91.4 x 72.4 mm, 15 parts

Commit message: Updated Code and Report
Parts:
- added REF**: PinSocket_2x08_P2.54mm_Vertical, Connector_PinSocket_2.54mm:PinSocket_2x08_P2.54mm_Vertical, F.Cu at (63.0, 64.8)
- added REF**: MountingHole_3mm, MountingHole:MountingHole_3mm, F.Cu at (21.1, 119.4)
- added REF**: MountingHole_3mm, MountingHole:MountingHole_3mm, F.Cu at (102.3, 119.4)
- added REF**: PinSocket_2x08_P2.54mm_Vertical, Connector_PinSocket_2.54mm:PinSocket_2x08_P2.54mm_Vertical, F.Cu at (40.1, 128.3)
- added REF**: PinSocket_1x06_P2.54mm_Vertical, Connector_PinSocket_2.54mm:PinSocket_1x06_P2.54mm_Vertical, F.Cu at (55.4, 95.3)
- added REF**: PinSocket_2x19_P2.54mm_Vertical, Connector_PinSocket_2.54mm:PinSocket_2x19_P2.54mm_Vertical, B.Cu at (90.9, 71.1)
- added REF**: MountingHole_3mm, MountingHole:MountingHole_3mm, F.Cu at (21.1, 64.8)
- added REF**: PinSocket_1x02_P2.54mm_Vertical, Connector_PinSocket_2.54mm:PinSocket_1x02_P2.54mm_Vertical, B.Cu at (61.7, 125.7)
- added REF**: PinSocket_2x19_P2.54mm_Vertical, Connector_PinSocket_2.54mm:PinSocket_2x19_P2.54mm_Vertical, B.Cu at (29.9, 71.1)
- added REF**: PinSocket_1x02_P2.54mm_Vertical, Connector_PinSocket_2.54mm:PinSocket_1x02_P2.54mm_Vertical, B.Cu at (55.4, 125.7)
- added REF**: PinSocket_1x02_P2.54mm_Vertical, Connector_PinSocket_2.54mm:PinSocket_1x02_P2.54mm_Vertical, B.Cu at (68.0, 125.7)
- added REF**: MountingHole_3mm, MountingHole:MountingHole_3mm, F.Cu at (102.3, 64.8)
- added REF**: PinSocket_1x06_P2.54mm_Vertical, Connector_PinSocket_2.54mm:PinSocket_1x06_P2.54mm_Vertical, F.Cu at (68.1, 95.3)
- added REF**: PinSocket_2x08_P2.54mm_Vertical, Connector_PinSocket_2.54mm:PinSocket_2x08_P2.54mm_Vertical, F.Cu at (83.3, 125.7)
Routing:
- net (no net): track 972.9 -> 1876.0 mm
Other:
- board size 91.4 x 72.4 mm -> 184.2 x 72.4 mm
- board text added: "EXT_PWR"

Commit message: Updated PCB, 3d Models, and some Code to fix mistakes.
Parts:
- removed the REF** at (63.0, 64.8)
- removed the REF** at (21.1, 119.4)
- removed the REF** at (102.3, 119.4)
- removed the REF** at (40.1, 128.3)
- removed the REF** at (55.4, 95.3)
- removed the REF** at (90.9, 71.1)
- removed the REF** at (21.1, 64.8)
- removed the REF** at (61.7, 125.7)
- removed the REF** at (29.9, 71.1)
- removed the REF** at (55.4, 125.7)
- removed the REF** at (68.0, 125.7)
- removed the REF** at (102.3, 64.8)
- removed the REF** at (68.1, 95.3)
- removed the REF** at (83.3, 125.7)
- moved REF** 43.7 mm to (85.8, 78.7)
- moved REF** 43.7 mm to (147.5, 53.4)
- moved REF** 43.7 mm to (136.6, 106.7)
- moved REF** 43.7 mm to (132.8, 66.0)
- moved REF** 43.7 mm to (128.4, 98.8)
- moved REF** 43.7 mm to (143.7, 98.8)
- moved REF** 43.7 mm to (108.1, 98.8)
- moved REF** 43.7 mm to (134.1, 78.7)
- moved REF** 43.7 mm to (116.3, 45.7)
- moved REF** 43.7 mm to (93.5, 109.2)
- moved REF** 43.7 mm to (125.2, 63.5)
- moved REF** 43.7 mm to (92.9, 98.8)
- moved REF** 43.7 mm to (118.3, 88.6)
- moved REF** 43.7 mm to (118.3, 108.9)
- moved REF** 20.5 mm to (106.2, 66.0)
Routing:
- net (no net): track 1876.0 -> 790.0 mm
Other:
- board size 184.2 x 72.4 mm -> 91.4 x 72.4 mm
- board text removed: "EXT_PWR"
